Commit message: Separate body from base_link and connect them with dummy_joint

File: robots/yamax.urdf (robot description, URDF)
Before this commit: robot yamax, 20 links, 19 joints
Links:
- added link body, mass 0.233; collision box size=0.05 0.11 0.094; visual box size=0.05 0.11 0.094
- link base_link: mass 0.233 -> None; geometry 
Joints:
- added joint dummy_joint: type fixed, parent base_link, child body
- joint neck: parent base_link -> body
- joint shoulder_right_x: parent base_link -> body

Commit message: Add inertial element to virtual links so that gazebo would recognize them correctly

File: robots/yamax.urdf (robot description, URDF)
Before this commit: robot yamax, 21 links, 20 joints
Links:
- link arm_left_1: mass 0.00914 -> 0.00457
- link arm_left_virtual: mass None -> 0.00457
- link arm_right_1: mass 0.00914 -> 0.00457
- link arm_right_virtual: mass None -> 0.00457

Commit message: Fix the connection between the backbone and the body

File: robots/yamax.urdf (robot description, URDF)
Before this commit: robot yamax, 21 links, 20 joints
Joints:
- joint backbone_1: parent base_link -> body

Commit message: Fix the connection between body and shoulder_right_x

File: robots/yamax.urdf (robot description, URDF)
Before this commit: robot yamax, 21 links, 20 joints
Joints:
- joint shoulder_left_x: parent base_link -> body
