Commit message: [WIP] Commit changes sent from @Nyanyan

File: robots/yamax.xacro (robot description, xacro)
@@ -5,26 +5,37 @@
   <xacro:include filename="$(cwd)/xacro/joint.xacro" />
   <xacro:include filename="$(cwd)/xacro/material.xacro" />
-  <xacro:link name="base_link" w="0.100" h="0.160" d="0.004" mass="0.207" x="0" y="0" z="0" material="Orange" has_imu="true" />
-  <xacro:link name="board" w="0.085" h="0.115" d="0.065" mass="0.220" x="0" y="0" z="0.0325" material="Black" />
-  <xacro:fixed_joint name="board" parent="base_link" child="board" z="0.004" />
-  <!-- hip_joint_*_p, knee_*, ankle_*_p joints are line symmetry -->
-  <!-- other joints are point symmetry                           -->
-  <xacro:fixed_joint name="hip_right" parent="base_link" child="hip_right" y="-0.051" z="-0.004" />
+  <link name="base_link" />
+  <xacro:link name="hip" w="0.090" h="0.150" d="0.004" mass="0.07061" x="0" y="0" z="0" material="Orange" has_imu="true" />
+  <xacro:link name="board" w="0.085" h="0.115" d="0.020" mass="0.1000" x="0" y="0" z="0.010" material="Black" />
+  <xacro:joint name="ignore_board" aname="board" parent="hip" child="board" z="0.004" axis="x" />
+  <xacro:joint name="ignore_hip_right" aname="ignore_hip_right" parent="hip" child="hip_right" y="-0.04325" z="-0.004" axis="x" />
   <xacro:link name="hip_right" w="0.0325" h="0.032" d="0.043" y="0" z="-0.0215" mass="0.0552" material="Black" />
-  <xacro:joint name="hip_joint_right_r" aname="K" parent="hip_right" child="virtual_hip_right" z="-0.030" axis="x" />
-  <xacro:virtual_link name="virtual_hip_right" w="0.01" h="0.01" d="0.01" z="-0.020" mass="0.0113" />
-  <xacro:joint name="hip_joint_right_p" aname="L" parent="virtual_hip_right" child="leg_right_1" z="-0.040" axis="y" />
-  <xacro:link name="leg_right_1" w="0.0325" h="0.032" d="0.043" z="-0.013" mass="0.0742" material="Black" />
+<!--  <xacro:joint name="hip_joint_right_r" aname="K" parent="hip_right" child="virtual_hip_right" z="-0.030" axis="x" />
+  <xacro:virtual_link name="virtual_hip_right" w="0.01" h="0.01" d="0.01" z="-0.020" mass="0.0113" /> -->
+  <xacro:joint name="hip_joint_right_p" aname="L" parent="hip_right" child="leg_right_1" z="-0.031" axis="y" />
+  <xacro:link name="leg_right_1" w="0.0325" h="0.032" d="0.043" z="-0.0415" mass="0.06772" material="Black" />
   <xacro:joint name="knee_right" aname="M" parent="leg_right_1" child="leg_right_2" z="-0.051" axis="y" />
-  <xacro:link name="leg_right_2" w="0.0325" h="0.032" d="0.043" z="-0.013" mass="0.0742" material="Black" />
-  <xacro:joint name="ankle_right_p" aname="N" parent="leg_right_2" child="leg_right_3" z="-0.051" axis="y" />
-  <xacro:link name="leg_right_3" w="0.0325" h="0.032" d="0.086" z="-0.034" mass="0.135" material="Black" />
-  <xacro:joint name="ankle_right_r" aname="O" parent="leg_right_3" child="foot_right" z="-0.065" axis="x" />
-  <xacro:link name="foot_right" w="0.094" h="0.064" d="0.013" z="-0.0275" mass="0.102" material="Orange" />
-  <xacro:fixed_joint name="hip_left" parent="base_link" child="hip_left" y="0.051" z="-0.004" yaw="${-pi}" />
+  <xacro:link name="leg_right_2" w="0.0325" h="0.032" d="0.043" z="-0.0385" mass="0.07270" material="Black" />
+<!--  <xacro:joint name="ankle_right_p" aname="N" parent="leg_right_2" child="leg_right_3" z="-0.051" axis="y" />
+  <xacro:link name="leg_right_3" w="0.0325" h="0.032" d="0.086" z="-0.034" mass="0.135" material="Black" /> -->
+  <xacro:joint name="ankle_right_r" aname="O" parent="leg_right_2" child="foot_right" z="-0.047.5" axis="x" />
+  <xacro:link name="foot_right" w="0.098" h="0.066" d="0.009" z="-0.0245" mass="0.05252" material="Orange" />
+  <xacro:joint name="ignore_hip_left" aname="ignore_hip_left" parent="hip" child="hip_left" y="0.04325" z="-0.004" axis="x" />
+  <xacro:link name="hip_left" w="0.0325" h="0.032" d="0.043" y="0" z="-0.0215" mass="0.0552" material="Black" />
+<!--  <xacro:joint name="hip_joint_right_r" aname="K" parent="hip_right" child="virtual_hip_right" z="-0.030" axis="x" />
+  <xacro:virtual_link name="virtual_hip_right" w="0.01" h="0.01" d="0.01" z="-0.020" mass="0.0113" /> -->
+  <xacro:joint name="hip_joint_left_p" aname="L" parent="hip_left" child="leg_left_1" z="-0.031" axis="y" />
+  <xacro:link name="leg_left_1" w="0.0325" h="0.032" d="0.043" z="-0.0415" mass="0.06772" material="Black" />
+  <xacro:joint name="knee_left" aname="M" parent="leg_left_1" child="leg_left_2" z="-0.051" axis="y" />
+  <xacro:link name="leg_left_2" w="0.0325" h="0.032" d="0.043" z="-0.0385" mass="0.07270" material="Black" />
+<!--  <xacro:joint name="ankle_right_p" aname="N" parent="leg_right_2" child="leg_right_3" z="-0.051" axis="y" />
+  <xacro:link name="leg_right_3" w="0.0325" h="0.032" d="0.086" z="-0.034" mass="0.135" material="Black" /> -->
+  <xacro:joint name="ankle_left_r" aname="O" parent="leg_left_2" child="foot_left" z="-0.047.5" axis="x" />
+  <xacro:link name="foot_left" w="0.098" h="0.066" d="0.009" z="-0.0245" mass="0.05252" material="Orange" />
+<!--  <xacro:joint name="ignore_hip_left" aname="ignore_hip_left" parent="hip" child="hip_left" y="0.051" z="-0.004" axis="x" />
   <xacro:link name="hip_left" w="0.0325" h="0.032" d="0.043" y="0" z="-0.0215" mass="0.0552" material="Black" />
   <xacro:joint name="hip_joint_left_r" aname="Q" parent="hip_left" child="virtual_hip_left" z="-0.030" axis="x" />
   <xacro:virtual_link name="virtual_hip_left" w="0.01" h="0.01" d="0.01" z="-0.020" mass="0.0113" />
-  <xacro:joint name="hip_joint_left_p" aname="R" parent="virtual_hip_left" child="leg_left_1" z="-0.040" yaw="${pi}" axis="y" />
+  <xacro:joint name="hip_joint_left_p" aname="R" parent="virtual_hip_left" child="leg_left_1" z="-0.040" axis="y" />
   <xacro:link name="leg_left_1" w="0.0325" h="0.032" d="0.043" z="-0.013" mass="0.0742" material="Black" />
   <xacro:joint name="knee_left" aname="S" parent="leg_left_1" child="leg_left_2" z="-0.051" axis="y" />
@@ -32,6 +43,11 @@
   <xacro:joint name="ankle_left_p" aname="T" parent="leg_left_2" child="leg_left_3" z="-0.051" axis="y" />
   <xacro:link name="leg_left_3" w="0.0325" h="0.032" d="0.086" z="-0.034" mass="0.135" material="Black" />
-  <xacro:joint name="ankle_left_r" aname="U" parent="leg_left_3" child="foot_left" z="-0.065" yaw="${-pi}" axis="x" />
+  <xacro:joint name="ankle_left_r" aname="U" parent="leg_left_3" child="foot_left" z="-0.065" axis="x" />
   <xacro:link name="foot_left" w="0.094" h="0.064" d="0.013" z="-0.0275" mass="0.102" material="Orange" />
+-->
+  <joint name="dummy_joint" type="fixed">
+    <parent link="base_link"/>
+    <child link="hip"/>
+  </joint>
   <gazebo>
     <plugin name="ground_truth" filename="libgazebo_ros_p3d.so">

Commit message: Fix: Fix relantions between base_link

File: robots/yamax.xacro (robot description, xacro)
@@ -5,49 +5,23 @@
   <xacro:include filename="$(cwd)/xacro/joint.xacro" />
   <xacro:include filename="$(cwd)/xacro/material.xacro" />
-  <link name="base_link" />
-  <xacro:link name="hip" w="0.090" h="0.150" d="0.004" mass="0.07061" x="0" y="0" z="0" material="Orange" has_imu="true" />
+  <xacro:link name="base_link" w="0.090" h="0.150" d="0.004" mass="0.07061" x="0" y="0" z="0" material="Orange" has_imu="true" />
   <xacro:link name="board" w="0.085" h="0.115" d="0.020" mass="0.1000" x="0" y="0" z="0.010" material="Black" />
-  <xacro:fixed_joint name="board" aname="board" parent="hip" child="board" z="0.004" axis="x" />
-  <xacro:fixed_joint name="hip_right" aname="ignore_hip_right" parent="hip" child="hip_right" y="-0.04325" z="-0.004" axis="x" />
+  <xacro:fixed_joint name="board" aname="board" parent="base_link" child="board" z="0.004" axis="x" />
+  <xacro:fixed_joint name="hip_right" aname="ignore_hip_right" parent="base_link" child="hip_right" y="-0.04325" z="-0.004" axis="x" />
   <xacro:link name="hip_right" w="0.0325" h="0.032" d="0.043" y="0" z="-0.0215" mass="0.0552" material="Black" />
-<!--  <xacro:joint name="hip_joint_right_r" aname="K" parent="hip_right" child="virtual_hip_right" z="-0.030" axis="x" />
-  <xacro:virtual_link name="virtual_hip_right" w="0.01" h="0.01" d="0.01" z="-0.020" mass="0.0113" /> -->
   <xacro:joint name="hip_joint_right_p" aname="L" parent="hip_right" child="leg_right_1" z="-0.031" axis="y" />
   <xacro:link name="leg_right_1" w="0.0325" h="0.032" d="0.043" z="-0.0415" mass="0.06772" material="Black" />
   <xacro:joint name="knee_right" aname="M" parent="leg_right_1" child="leg_right_2" z="-0.051" axis="y" />
   <xacro:link name="leg_right_2" w="0.0325" h="0.032" d="0.043" z="-0.0385" mass="0.07270" material="Black" />
-<!--  <xacro:joint name="ankle_right_p" aname="N" parent="leg_right_2" child="leg_right_3" z="-0.051" axis="y" />
-  <xacro:link name="leg_right_3" w="0.0325" h="0.032" d="0.086" z="-0.034" mass="0.135" material="Black" /> -->
   <xacro:joint name="ankle_right_r" aname="O" parent="leg_right_2" child="foot_right" z="-0.047.5" axis="x" />
   <xacro:link name="foot_right" w="0.098" h="0.066" d="0.009" z="-0.0245" mass="0.05252" material="Orange" />
-  <xacro:fixed_joint name="hip_left" aname="ignore_hip_left" parent="hip" child="hip_left" y="0.04325" z="-0.004" axis="x" />
+  <xacro:fixed_joint name="hip_left" aname="ignore_hip_left" parent="base_link" child="hip_left" y="0.04325" z="-0.004" axis="x" />
   <xacro:link name="hip_left" w="0.0325" h="0.032" d="0.043" y="0" z="-0.0215" mass="0.0552" material="Black" />
-<!--  <xacro:joint name="hip_joint_right_r" aname="K" parent="hip_right" child="virtual_hip_right" z="-0.030" axis="x" />
-  <xacro:virtual_link name="virtual_hip_right" w="0.01" h="0.01" d="0.01" z="-0.020" mass="0.0113" /> -->
   <xacro:joint name="hip_joint_left_p" aname="L" parent="hip_left" child="leg_left_1" z="-0.031" axis="y" />
   <xacro:link name="leg_left_1" w="0.0325" h="0.032" d="0.043" z="-0.0415" mass="0.06772" material="Black" />
   <xacro:joint name="knee_left" aname="M" parent="leg_left_1" child="leg_left_2" z="-0.051" axis="y" />
   <xacro:link name="leg_left_2" w="0.0325" h="0.032" d="0.043" z="-0.0385" mass="0.07270" material="Black" />
-<!--  <xacro:joint name="ankle_right_p" aname="N" parent="leg_right_2" child="leg_right_3" z="-0.051" axis="y" />
-  <xacro:link name="leg_right_3" w="0.0325" h="0.032" d="0.086" z="-0.034" mass="0.135" material="Black" /> -->
   <xacro:joint name="ankle_left_r" aname="O" parent="leg_left_2" child="foot_left" z="-0.047.5" axis="x" />
   <xacro:link name="foot_left" w="0.098" h="0.066" d="0.009" z="-0.0245" mass="0.05252" material="Orange" />
-<!--  <xacro:joint name="ignore_hip_left" aname="ignore_hip_left" parent="hip" child="hip_left" y="0.051" z="-0.004" axis="x" />
-  <xacro:link name="hip_left" w="0.0325" h="0.032" d="0.043" y="0" z="-0.0215" mass="0.0552" material="Black" />
-  <xacro:joint name="hip_joint_left_r" aname="Q" parent="hip_left" child="virtual_hip_left" z="-0.030" axis="x" />
-  <xacro:virtual_link name="virtual_hip_left" w="0.01" h="0.01" d="0.01" z="-0.020" mass="0.0113" />
-  <xacro:joint name="hip_joint_left_p" aname="R" parent="virtual_hip_left" child="leg_left_1" z="-0.040" axis="y" />
-  <xacro:link name="leg_left_1" w="0.0325" h="0.032" d="0.043" z="-0.013" mass="0.0742" material="Black" />
-  <xacro:joint name="knee_left" aname="S" parent="leg_left_1" child="leg_left_2" z="-0.051" axis="y" />
-  <xacro:link name="leg_left_2" w="0.0325" h="0.032" d="0.043" z="-0.013" mass="0.0742" material="Black" />
-  <xacro:joint name="ankle_left_p" aname="T" parent="leg_left_2" child="leg_left_3" z="-0.051" axis="y" />
-  <xacro:link name="leg_left_3" w="0.0325" h="0.032" d="0.086" z="-0.034" mass="0.135" material="Black" />
-  <xacro:joint name="ankle_left_r" aname="U" parent="leg_left_3" child="foot_left" z="-0.065" axis="x" />
-  <xacro:link name="foot_left" w="0.094" h="0.064" d="0.013" z="-0.0275" mass="0.102" material="Orange" />
--->
-  <joint name="dummy_joint" type="fixed">
-    <parent link="base_link"/>
-    <child link="hip"/>
-  </joint>
   <gazebo>
     <plugin name="ground_truth" filename="libgazebo_ros_p3d.so">
