Commit message: Remove soft_{cfm, erp}
beacuse they has no effect:scream:
http://answers.gazebosim.org/question/13807/is-soft_cfm-and-soft_erp-utilized-by-ode/

File: xacro/config/link.xacro (robot description, xacro)
@@ -5,6 +5,4 @@
   <xacro:property name="kp" value="100000000000.0" />
   <xacro:property name="kd" value="1000000000.0" />
-  <xacro:property name="soft_erp" value="0.8" />
-  <xacro:property name="soft_cfm" value="0.2" />
   <xacro:property name="max_vel" value="0.001" />
   <xacro:property name="min_depth" value="0.00001" />

File: xacro/link.xacro (robot description, xacro)
@@ -39,6 +39,4 @@
           <contact>
             <ode>
-              <soft_cfm>${config.link.soft_cfm}</soft_cfm>
-              <soft_erp>${config.link.soft_erp}</soft_erp>
               <kp>${config.link.kp}</kp>
               <kd>${config.link.kd}</kd>
@@ -47,6 +45,4 @@
             </ode>
             <bullet>
-              <soft_cfm>${config.link.soft_cfm}</soft_cfm>
-              <soft_erp>${config.link.soft_erp}</soft_erp>
               <kp>${config.link.kp}</kp>
               <kd>${config.link.kd}</kd>

Commit message: Reduce max_vel

File: xacro/config/link.xacro (robot description, xacro)
@@ -5,5 +5,5 @@
   <xacro:property name="kp" value="100000000000.0" />
   <xacro:property name="kd" value="1000000000.0" />
-  <xacro:property name="max_vel" value="0.001" />
+  <xacro:property name="max_vel" value="0.0001" />
   <xacro:property name="min_depth" value="0.00001" />
 </robot>

Commit message: Adjust parameters and finally be able to stand correctly

File: xacro/config/link.xacro (robot description, xacro)
@@ -1,9 +1,9 @@
 <?xml version="1.0"?>
 <robot xmlns:xacro="http://ros.org/wiki/xacro">
-  <xacro:property name="friction1" value="0.61" />
-  <xacro:property name="friction2" value="0.61" />
-  <xacro:property name="kp" value="100000000000.0" />
-  <xacro:property name="kd" value="1000000000.0" />
-  <xacro:property name="max_vel" value="0.0001" />
+  <xacro:property name="friction1" value="100" />
+  <xacro:property name="friction2" value="50" />
+  <xacro:property name="kp" value="1e+8" />
+  <xacro:property name="kd" value="1.0" />
+  <xacro:property name="max_vel" value="0.1" />
   <xacro:property name="min_depth" value="0.00001" />
 </robot>

Commit message: Adjust link parameters

File: xacro/config/link.xacro (robot description, xacro)
@@ -1,9 +1,9 @@
 <?xml version="1.0"?>
 <robot xmlns:xacro="http://ros.org/wiki/xacro">
-  <xacro:property name="friction1" value="100" />
-  <xacro:property name="friction2" value="50" />
-  <xacro:property name="kp" value="1e+8" />
-  <xacro:property name="kd" value="1.0" />
+  <xacro:property name="friction1" value="0.4" />
+  <xacro:property name="friction2" value="0.4" />
+  <xacro:property name="kp" value="1e+6" />
+  <xacro:property name="kd" value="1e-10" />
   <xacro:property name="max_vel" value="0.1" />
-  <xacro:property name="min_depth" value="0.00001" />
+  <xacro:property name="min_depth" value="0.1" />
 </robot>
