Commit message: Now the robot can stand with two legs, to enable ODE instaed of bullet

File: xacro/config/joint.xacro (robot description, xacro)
@@ -3,9 +3,9 @@
   <xacro:property name="lower" value="-1.5708" />
   <xacro:property name="upper" value="1.5708" />
-  <xacro:property name="effort" value="10" />
-  <xacro:property name="velocity" value="10" />
+  <xacro:property name="effort" value="300" />
+  <xacro:property name="velocity" value="1.17" />
   <xacro:property name="hardware_interface" value="hardware_interface/PositionJointInterface" />
   <xacro:property name="transmission_interface" value="transmission_interface/SimpleTransmission" />
   <xacro:property name="transmission_suffix" value="_transmission" />
-  <xacro:property name="mechanical_reduction" value="50" />
+  <xacro:property name="mechanical_reduction" value="1.0" />
 </robot>

File: xacro/config/link.xacro (robot description, xacro)
@@ -3,5 +3,9 @@
   <xacro:property name="friction1" value="0.61" />
   <xacro:property name="friction2" value="0.61" />
-  <xacro:property name="kp" value="1000000.0" />
-  <xacro:property name="kd" value="1.0" />
+  <xacro:property name="kp" value="100000000000.0" />
+  <xacro:property name="kd" value="1000000000.0" />
+  <xacro:property name="soft_erp" value="0.8" />
+  <xacro:property name="soft_cfm" value="0.2" />
+  <xacro:property name="max_vel" value="0.001" />
+  <xacro:property name="min_depth" value="0.00001" />
 </robot>

File: xacro/link.xacro (robot description, xacro)
@@ -28,4 +28,8 @@
         <surface>
           <friction>
+            <ode>
+              <mu>${config.link.friction1}</mu>
+              <mu2>${config.link.friction2}</mu2>
+            </ode>
             <bullet>
               <friction>${config.link.friction1}</friction>
@@ -34,5 +38,15 @@
           </friction>
           <contact>
+            <ode>
+              <soft_cfm>${config.link.soft_cfm}</soft_cfm>
+              <soft_erp>${config.link.soft_erp}</soft_erp>
+              <kp>${config.link.kp}</kp>
+              <kd>${config.link.kd}</kd>
+              <max_vel>${config.link.max_vel}</max_vel>
+              <min_depth>${config.link.min_depth}</min_depth>
+            </ode>
             <bullet>
+              <soft_cfm>${config.link.soft_cfm}</soft_cfm>
+              <soft_erp>${config.link.soft_erp}</soft_erp>
               <kp>${config.link.kp}</kp>
               <kd>${config.link.kd}</kd>

Commit message: Reduce effort of joint

File: xacro/config/joint.xacro (robot description, xacro)
@@ -3,5 +3,5 @@
   <xacro:property name="lower" value="-1.5708" />
   <xacro:property name="upper" value="1.5708" />
-  <xacro:property name="effort" value="300" />
+  <xacro:property name="effort" value="3" />
   <xacro:property name="velocity" value="1.17" />
   <xacro:property name="hardware_interface" value="hardware_interface/PositionJointInterface" />

Commit message: Fix: Set upper and lower bounds based on pi

File: xacro/config/joint.xacro (robot description, xacro)
@@ -1,6 +1,6 @@
 <?xml version="1.0"?>
 <robot xmlns:xacro="http://ros.org/wiki/xacro">
-  <xacro:property name="lower" value="-1.5708" />
-  <xacro:property name="upper" value="1.5708" />
+  <xacro:property name="lower" value="${-pi / 2}" />
+  <xacro:property name="upper" value="${ pi / 2}" />
   <xacro:property name="effort" value="3" />
   <xacro:property name="velocity" value="1.17" />

Commit message: Fix: Set effort and velocity limit correctly

File: xacro/config/joint.xacro (robot description, xacro)
@@ -3,6 +3,9 @@
   <xacro:property name="lower" value="${-pi / 2}" />
   <xacro:property name="upper" value="${ pi / 2}" />
-  <xacro:property name="effort" value="3" />
-  <xacro:property name="velocity" value="1.17" />
+  <!-- https://kondo-robot.com/product/krs-4031hv-ics -->
+  <!-- 13.0kgf・cm -->
+  <!-- 0.16s/60°   -->
+  <xacro:property name="effort" value="13.0" />
+  <xacro:property name="velocity" value="${pi / 3 / 0.16}" />
   <xacro:property name="hardware_interface" value="hardware_interface/PositionJointInterface" />
   <xacro:property name="transmission_interface" value="transmission_interface/SimpleTransmission" />

Commit message: Fix: Fix joint bounds

File: xacro/config/joint.xacro (robot description, xacro)
@@ -1,7 +1,8 @@
 <?xml version="1.0"?>
 <robot xmlns:xacro="http://ros.org/wiki/xacro">
-  <xacro:property name="lower" value="${-pi / 2}" />
-  <xacro:property name="upper" value="${ pi / 2}" />
   <!-- https://kondo-robot.com/product/krs-4031hv-ics -->
+  <!-- 270° -->
+  <xacro:property name="lower" value="${-2 * pi / 3}" />
+  <xacro:property name="upper" value="${ 2 * pi / 3}" />
   <!-- 13.0kgf・cm -->
   <!-- 0.16s/60°   -->

Commit message: Fix: Convert kgfcm to Nm

File: xacro/config/joint.xacro (robot description, xacro)
@@ -7,5 +7,5 @@
   <!-- 13.0kgf・cm -->
   <!-- 0.16s/60°   -->
-  <xacro:property name="effort" value="13.0" />
+  <xacro:property name="effort" value="${13.0 / 0.09807}" />
   <xacro:property name="velocity" value="${pi / 3 / 0.16}" />
   <xacro:property name="hardware_interface" value="hardware_interface/PositionJointInterface" />
